Commit message: Added Section 2 (Cleaned)

File: samples/ramp.urdf (robot description, URDF)
Before this commit: robot box, 3 links, 2 joints
Links:
- link base: mass 300.0 -> 1000.0; geometry collision box size=4 2 1.5; visual box size=4 2 1.5
- link left_ramp: geometry collision box size=3.35 2.0 0.02; visual box size=3.35 2.0 0.02
- link right_ramp: geometry collision box size=3.35 2.0 0.02; visual box size=3.35 2.0 0.02
Joints:
- joint base2leftramp: origin xyz=-2 0 1 rpy=0.0 -0.5880 0.0 -> xyz=-2 0 0.75 rpy=0.0 -0.46 0.0
- joint base2rightramp: origin xyz=2 0 1 rpy=0.0 0.588 0.0 -> xyz=2 0 0.75 rpy=0.0 0.4636 0.0
