Commit message: Stable Version with Section 3

File: samples/barrier.urdf (robot description, URDF)
Before this commit: robot box, 2 links, 1 joints
Links:
- link base: mass 90.0 -> 0.0
Joints:
- joint base2stick: limit lower=0 upper=1.58 effort=10.0 velocity=10.0 -> lower=0 upper=1.58 effort=5.0 velocity=5.0

Commit message: Entrega

File: samples/barrier.urdf (robot description, URDF)
Before this commit: robot box, 2 links, 1 joints
Joints:
- joint base2stick: limit lower=0 upper=1.58 effort=5.0 velocity=5.0 -> lower=0 upper=1.58 effort=100.0 velocity=60.0
